File: hw-microdiff.sch (KiCad schematic (older format))
At the start: 26 parts, among them J1 RJ45, J2 JST 1x8, J3 Screw_Terminal_01x02, SW1 SW_DIP_x02, U1 5V, U2 RS-485 IC, U3 3.3V

Commit message: Finish PCB routing for v.04
Parts:
- removed C2: 10uF, Capacitor_SMD:CP_Elec_5x5.3, symbol Device:CP
- removed H1: M3_MountingHole_Pad, MountingHole:MountingHole_3.2mm_M3_Pad_Via, symbol Mechanical:MountingHole_Pad
- removed J1: RJ45, Connector_RJ:RJ45_Amphenol_54602-x08_Horizontal, symbol Connector:RJ45
- removed SW1: SW_DIP_x02, Button_Switch_THT:SW_DIP_SPSTx02_Slide_9.78x7.26mm_W7.62mm_P2.54mm, symbol Switch:SW_DIP_x02
- removed U2: RS-485 IC, Package_DIP:DIP-8_W7.62mm_Socket, symbol 2021-04-08_14-20-24:max3088cpa+
- added C4: 0.1uF 50V, Capacitor_SMD:C_0603_1608Metric, symbol Device:C
- added D2: Blue LED, LED_SMD:LED_0603_1608Metric, symbol Device:LED
- added J3: 8P8C, Connector_RJ:RJ45_Hanrun_HR911105A, symbol Connector:8P8C_Shielded
- added JP1: GND EN, Connector_PinHeader_2.54mm:PinHeader_1x02_P2.54mm_Vertical, symbol Device:Jumper_NO_Small
- added JP3: drive EN, Button_Switch_THT:SW_DIP_SPSTx01_Slide_9.78x4.72mm_W7.62mm_P2.54mm, symbol Device:Jumper_NO_Small
- added R8: 10K, Resistor_SMD:R_0805_2012Metric, symbol Device:R
- added U3: RS-485, Package_SO:SOIC-8_3.9x4.9mm_P1.27mm, symbol Interface_UART:SP3485EN
- C1: value 0.1uF -> 0.1uF 50V; footprint Capacitor_SMD:C_0805_2012Metric_Pad1.18x1.45mm_HandSolder -> Capacitor_SMD:C_0603_1608Metric; LCSC (none) -> C14663; LCSC Part C49678 -> C14663
- C2: renamed from C3; value 22uF -> 22uF 10V; footprint Capacitor_SMD:CP_Elec_5x5.3 -> Capacitor_SMD:C_1206_3216Metric; symbol Device:CP -> Device:C; LCSC (none) -> C5672; LCSC Part C249477 -> C5672
- C3: renamed from C4; value 10uF -> 22uF 10V; footprint Capacitor_SMD:C_0805_2012Metric_Pad1.18x1.45mm_HandSolder -> Capacitor_SMD:C_1206_3216Metric; LCSC (none) -> C5672; LCSC Part C15850 -> C5672
- C5: value 10uF -> 10uF 10V; footprint Capacitor_SMD:C_0805_2012Metric_Pad1.18x1.45mm_HandSolder -> Capacitor_SMD:C_0603_1608Metric; LCSC (none) -> C19702; LCSC Part C15850 -> C19702
- D1: value D_Schottky -> Diode 40V/3A; footprint Diode_SMD:D_SMA_Handsoldering -> Diode_SMD:D_SMA; LCSC (none) -> C8678; LCSC Part C22452 -> C8678; Part # (none) -> SS34
- F1: value Polyfuse -> Fuse 24V/1A; footprint Fuse:Fuse_Bourns_MF-RHT050 -> Fuse:Fuse_1206_3216Metric; symbol Device:Polyfuse -> Device:Fuse; LCSC (none) -> C910830; LCSC Part (none) -> C910830; Part # (none) -> BSMD1206-100-24V
- H2, H3, H4: value M3_MountingHole_Pad -> M2_MountingHole; footprint MountingHole:MountingHole_3.2mm_M3_Pad_Via -> MountingHole:MountingHole_2.2mm_M2_ISO14580_Pad; symbol Mechanical:MountingHole_Pad -> Mechanical:MountingHole
- J1: renamed from J3; value Screw_Terminal_01x02 -> Power Input; footprint TerminalBlock_Phoenix:TerminalBlock_Phoenix_PT-1,5-2-5.0-H_1x02_P5.00mm_Horizontal -> Connector_PinHeader_2.54mm:PinHeader_1x02_P2.54mm_Vertical; symbol Connector:Screw_Terminal_01x02 -> Connector_Generic:Conn_01x02; LCSC Part C557685 -> (none)
- J2: value JST 1x8 -> Header 2x4P; footprint Connector_JST:JST_XH_B8B-XH-A_1x08_P2.50mm_Vertical -> Connector_PinSocket_2.54mm:PinSocket_2x04_P2.54mm_Vertical; symbol Connector_Generic:Conn_01x08 -> Connector_Generic:Conn_02x04_Odd_Even; LCSC Part C5663 -> (none)
- JP2: renamed from JP1; value JUMPER -> VIN EN; footprint Connector_PinHeader_2.54mm:PinHeader_1x03_P2.54mm_Vertical -> Connector_PinHeader_2.54mm:PinHeader_1x02_P2.54mm_Vertical
- R1: value 120R -> 220R; footprint Resistor_THT:R_Axial_DIN0207_L6.3mm_D2.5mm_P10.16mm_Horizontal -> Resistor_SMD:R_0805_2012Metric; LCSC (none) -> C17557; LCSC Part (none) -> C17557
- R2, R4: footprint Resistor_SMD:R_0805_2012Metric_Pad1.20x1.40mm_HandSolder -> Resistor_SMD:R_0805_2012Metric
- R3: value 10K -> 20K; LCSC Part C17414 -> (none)
- R5: value 10K -> 120R; footprint Resistor_SMD:R_0805_2012Metric_Pad1.20x1.40mm_HandSolder -> Resistor_THT:R_Axial_DIN0207_L6.3mm_D2.5mm_P10.16mm_Horizontal; LCSC (none) -> C17437; LCSC Part C17414 -> (none)
- R6: value 20K -> 10K; footprint Resistor_SMD:R_0805_2012Metric_Pad1.20x1.40mm_HandSolder -> Resistor_SMD:R_0805_2012Metric; LCSC Part C4328 -> C17414
- R7: LCSC Part C4328 -> (none)
- U1: value 5V -> 5V/1A; footprint Converter_DCDC:Converter_DCDC_RECOM_R-78E-0.5_THT -> Package_TO_SOT_SMD:SOT-223; symbol Regulator_Switching:R-78E5.0-1.0 -> Regulator_Linear:AMS1117-5.0; LCSC (none) -> C6187; LCSC Part (none) -> C6187; Part # (none) -> AMS1117-5.0
- U2: renamed from U3; value 3.3V -> 3.3V/1A; LCSC (none) -> C6186; Part # (none) -> AMS1117-3.3
Connections:
- net labels added: 3V3, 5V, DE_RE, VSS, a1, b1
- net labels removed: A, B, DE, FUSE, PWR, RE, VCC
- wire segments 87 -> 85
Other:
- note added: "*Notes:*\n\n VIN / GND enable power through 8P8C connectors\n\n*Resistor Specifications:*\n\n 120R, ±1% 118.8Ω - 121.2Ω, 0805, 1/8W (125mW)\n 220R, ±1% 217.8Ω - 222.2Ω, 0805, 1/8W (125mW)\n 10K, ±1% 9.9kΩ - 10.1kΩ, 0805, 1/8W (125mW)\n 20K, ±1% 19.8kΩ - 20.2kΩ, 0805, 1/8W (125mW)"
- note added: "DC-DC 3.3V"
- note added: "DC-DC 5V"
- note added: "DNP"
- note added: "Output"
- note added: "VIN 6.5V-12V"
- note added: "biasing"
- note removed: "Connectors"
- note removed: "Input Voltage Regulators"
- moved on the sheet: C1, C3, D1, J2, JP2, U1, U2

Commit message: Minor layout corrections:   - Add test pads on back of PCB   - Remove 10K pullup   - Adjust silkscreens   - Update to KiCad 6.0   - Add 3D model for RJ45 connector   - Add VDD pin for unprotected VIN   - Add open jumpers and remove DIP switch   - Connect RJ45 shield and H2 mounting hole to Earth, not ground
Parts:
- added TP1: TP_VIN, TestPoint:TestPoint_Pad_1.5x1.5mm, symbol Connector:TestPoint
- added TP10: TP_B1, TestPoint:TestPoint_Pad_D1.5mm, symbol Connector:TestPoint
- added TP2, TP8: TP_GND, TestPoint:TestPoint_Pad_1.5x1.5mm, symbol Connector:TestPoint
- added TP3: TP_5V, TestPoint:TestPoint_Pad_1.5x1.5mm, symbol Connector:TestPoint
- added TP4: TP_3V3, TestPoint:TestPoint_Pad_1.5x1.5mm, symbol Connector:TestPoint
- added TP5: TP_RO, TestPoint:TestPoint_Pad_D1.5mm, symbol Connector:TestPoint
- added TP6: TP_DI, TestPoint:TestPoint_Pad_D1.5mm, symbol Connector:TestPoint
- added TP7: TP_DE_RE, TestPoint:TestPoint_Pad_D1.5mm, symbol Connector:TestPoint
- added TP9: TP_A1, TestPoint:TestPoint_Pad_D1.5mm, symbol Connector:TestPoint
- R4: value 10K -> 4K7; LCSC Part C17414 -> C17673
Connections:
- wire segments 85 -> 95
Other:
- note added: "*Notes:*\n\n VIN / GND enable power through 8P8C connectors\n\n*Resistor Specifications:*\n\n 120R, ±1% 118.8Ω - 121.2Ω, 0805, 1/8W (125mW)\n 220R, ±1% 217.8Ω - 222.2Ω, 0805, 1/8W (125mW)\n 4.7K, ±1% 4.653kΩ - 4.747kΩ, 0805, 1/8W (125mW)\n 10K, ±1% 9.9kΩ - 10.1kΩ, 0805, 1/8W (125mW)\n 20K, ±1% 19.8kΩ - 20.2kΩ, 0805, 1/8W (125mW)"
- note added: "Test Points"
- note removed: "*Notes:*\n\n VIN / GND enable power through 8P8C connectors\n\n*Resistor Specifications:*\n\n 120R, ±1% 118.8Ω - 121.2Ω, 0805, 1/8W (125mW)\n 220R, ±1% 217.8Ω - 222.2Ω, 0805, 1/8W (125mW)\n 10K, ±1% 9.9kΩ - 10.1kΩ, 0805, 1/8W (125mW)\n 20K, ±1% 19.8kΩ - 20.2kΩ, 0805, 1/8W (125mW)"
Changed lines of the file:
@@
 Wire Notes Line
 	5600 6400 5600 4200
-Text Notes 5750 5050 0    50   Italic 0
-*Notes:*\n\n   VIN / GND enable power through 8P8C connectors\n\n*Resistor Specifications:*\n\n  120R, ±1% 118.8Ω - 121.2Ω, 0805, 1/8W (125mW)\n  220R, ±1% 217.8Ω - 222.2Ω, 0805, 1/8W (125mW)\n  10K, ±1% 9.9kΩ - 10.1kΩ, 0805, 1/8W (125mW)\n  20K, ±1% 19.8kΩ - 20.2kΩ, 0805, 1/8W (125mW)
+Text Notes 5750 5150 0    50   Italic 0
+*Notes:*\n\n   VIN / GND enable power through 8P8C connectors\n\n*Resistor Specifications:*\n\n  120R, ±1% 118.8Ω - 121.2Ω, 0805, 1/8W (125mW)\n  220R, ±1% 217.8Ω - 222.2Ω, 0805, 1/8W (125mW)\n  4.7K, ±1% 4.653kΩ - 4.747kΩ, 0805, 1/8W (125mW)\n  10K, ±1% 9.9kΩ - 10.1kΩ, 0805, 1/8W (125mW)\n  20K, ±1% 19.8kΩ - 20.2kΩ, 0805, 1/8W (125mW)
 Wire Notes Line
 	5700 4200 7950 4200
 Wire Notes Line
-	5700 5100 7950 5100
+	5700 5250 7950 5250
 $Comp
 L Interface_UART:SP3485EN U3
@@
 AR Path="/63E575AB/6311FF2C" Ref="R?"  Part="1"
 F 0 "R4" V 1100 5050 50  0000 L CNN
-F 1 "10K" V 1200 5030 50  0000 L CNN
+F 1 "4K7" V 1200 5030 50  0000 L CNN
 F 2 "Resistor_SMD:R_0805_2012Metric" V 1130 5100 50  0001 C CNN
 F 3 "~" H 1200 5100 50  0001 C CNN
 F 4 "" H 1200 5100 50  0001 C CNN "LCSC"
 F 5 "" H 1200 5100 50  0001 C CNN "LCSC Part #"
-F 6 "C17414" H 1200 5100 50  0001 C CNN "LCSC Part"
+F 6 "C17673" H 1200 5100 50  0001 C CNN "LCSC Part"
 	1    1200 5100
 	0    1    1    0
@@
 Wire Notes Line
 	700  7400 700  6550
-Wire Notes Line
-	7950 4200 7950 5100
-Wire Notes Line
-	5700 4200 5700 5100
+Text Label 3100 6950 0    50   ~ 0
+5V
+$Comp
+L Connector:TestPoint TP2
+U 1 1 62FA4E67
+P 2650 7250
+F 0 "TP2" H 2708 7368 50  0000 L CNN
+F 1 "TP_GND" H 2708 7277 50  0000 L CNN
+F 2 "TestPoint:TestPoint_Pad_1.5x1.5mm" H 2850 7250 50  0001 C CNN
+F 3 "~" H 2850 7250 50  0001 C CNN
+	1    2650 7250
+	1    0    0    -1
+$EndComp
+Text Label 2450 7250 0    50   ~ 0
+GND
+Text Label 4150 4850 0    50   ~ 0
+GND
+Wire Wire Line
+	2450 7250 2650 7250
+$Comp
+L Connector:TestPoint TP1
+U 1 1 62FBC60D
+P 2650 6950
+F 0 "TP1" H 2708 7068 50  0000 L CNN
+F 1 "TP_VIN" H 2708 6977 50  0000 L CNN
+F 2 "TestPoint:TestPoint_Pad_1.5x1.5mm" H 2850 6950 50  0001 C CNN
+F 3 "~" H 2850 6950 50  0001 C CNN
+	1    2650 6950
+	1    0    0    -1
+$EndComp
+Text Label 2450 6950 0    50   ~ 0
+VIN
+Wire Wire Line
+	2450 6950 2650 6950
+Wire Wire Line
+	3700 7250 3850 7250
+Text Label 3700 7250 0    50   ~ 0
+DI
+$Comp
+L Connector:TestPoint TP6
+U 1 1 62F9C2EF
+P 3850 7250
+F 0 "TP6" H 3908 7368 50  0000 L CNN
+F 1 "TP_DI" H 3908 7277 50  0000 L CNN
+F 2 "TestPoint:TestPoint_Pad_D1.5mm" H 4050 7250 50  0001 C CNN
+F 3 "~" H 4050 7250 50  0001 C CNN
+	1    3850 7250
+	1    0    0    -1
+$EndComp
+Wire Wire Line
+	4300 6950 4550 6950
+Text Label 4300 6950 0    50   ~ 0
+DE_RE
+$Comp
+L Connector:TestPoint TP7
+U 1 1 62F794B2
+P 4550 6950
+F 0 "TP7" H 4608 7068 50  0000 L CNN
+F 1 "TP_DE_RE" H 4608 6977 50  0000 L CNN
+F 2 "TestPoint:TestPoint_Pad_D1.5mm" H 4750 6950 50  0001 C CNN
+F 3 "~" H 4750 6950 50  0001 C CNN
+	1    4550 6950
+	1    0    0    -1
+$EndComp
+Wire Wire Line
+	3700 6950 3850 6950
+Text Label 3700 6950 0    50   ~ 0
+RO
+$Comp
+L Connector:TestPoint TP5
+U 1 1 62F6DF61
+P 3850 6950
+F 0 "TP5" H 3908 7068 50  0000 L CNN
+F 1 "TP_RO" H 3908 6977 50  0000 L CNN
+F 2 "TestPoint:TestPoint_Pad_D1.5mm" H 4050 6950 50  0001 C CNN
+F 3 "~" H 4050 6950 50  0001 C CNN
+	1    3850 6950
+	1    0    0    -1
+$EndComp
+Wire Wire Line
+	3100 7250 3250 7250
+Text Label 3100 7250 0    50   ~ 0
+3V3
+$Comp
+L Connector:TestPoint TP4
+U 1 1 62F6AB72
+P 3250 7250
+F 0 "TP4" H 3308 7368 50  0000 L CNN
+F 1 "TP_3V3" H 3308 7277 50  0000 L CNN
+F 2 "TestPoint:TestPoint_Pad_1.5x1.5mm" H 3450 7250 50  0001 C CNN
+F 3 "~" H 3450 7250 50  0001 C CNN
+	1    3250 7250
+	1    0    0    -1
+$EndComp
+Wire Wire Line
+	3100 6950 3250 6950
+$Comp
+L Connector:TestPoint TP3
+U 1 1 62F6119B
+P 3250 6950
+F 0 "TP3" H 3308 7068 50  0000 L CNN
+F 1 "TP_5V" H 3308 6977 50  0000 L CNN
+F 2 "TestPoint:TestPoint_Pad_1.5x1.5mm" H 3450 6950 50  0001 C CNN
+F 3 "~" H 3450 6950 50  0001 C CNN
+	1    3250 6950
+	1    0    0    -1
+$EndComp
+$Comp
+L Connector:TestPoint TP8
+U 1 1 6301059D
+P 4550 7250
+F 0 "TP8" H 4608 7368 50  0000 L CNN
+F 1 "TP_GND" H 4608 7277 50  0000 L CNN
+F 2 "TestPoint:TestPoint_Pad_1.5x1.5mm" H 4750 7250 50  0001 C CNN
+F 3 "~" H 4750 7250 50  0001 C CNN
+	1    4550 7250
+	1    0    0    -1
+$EndComp
+Text Label 4350 7250 0    50   ~ 0
+GND
+Wire Wire Line
+	4350 7250 4550 7250
+Wire Notes Line
+	5700 4200 5700 5250
+Wire Notes Line
+	7950 4200 7950 5250
+Wire Wire Line
+	5100 6950 5250 6950
+Text Label 5100 6950 0    50   ~ 0
+a1
+$Comp
+L Connector:TestPoint TP9
+U 1 1 63070A07
+P 5250 6950
+F 0 "TP9" H 5308 7068 50  0000 L CNN
+F 1 "TP_A1" H 5308 6977 50  0000 L CNN
+F 2 "TestPoint:TestPoint_Pad_D1.5mm" H 5450 6950 50  0001 C CNN
+F 3 "~" H 5450 6950 50  0001 C CNN
+	1    5250 6950
+	1    0    0    -1
+$EndComp
+Wire Wire Line
+	5100 7250 5250 7250
+Text Label 5100 7250 0    50   ~ 0
+b1
+$Comp
+L Connector:TestPoint TP10
+U 1 1 630751F1
+P 5250 7250
+F 0 "TP10" H 5308 7368 50  0000 L CNN
+F 1 "TP_B1" H 5308 7277 50  0000 L CNN
+F 2 "TestPoint:TestPoint_Pad_D1.5mm" H 5450 7250 50  0001 C CNN
+F 3 "~" H 5450 7250 50  0001 C CNN
+	1    5250 7250
+	1    0    0    -1
+$EndComp
+Wire Notes Line
+	2350 6550 2350 7400
+Wire Notes Line
+	2350 7400 5600 7400
+Wire Notes Line
+	5600 7400 5600 6550
+Wire Notes Line
+	5600 6550 2350 6550
+Text Notes 2400 6650 0    50   ~ 0
+Test Points
 $EndSCHEMATC
